Commit message: fix: correct MarsRover steering pivots and joint frames

File: urdf/mars.urdf (robot description, URDF)
Before this commit: robot tianrover_mars, 21 links, 20 joints
Links:
- added link body_top_link, mass 0.776301461341526; collision mesh filename=package://tianbot_description/meshes/base_footprint_link.STL; visual mesh filename=package://tianbot_description/meshes/base_footprint_link.STL
- link base_footprint: mass 0.776301461341526 -> None; geometry 
Joints:
- added joint body_top_joint: type fixed, parent base_link, child body_top_link, origin xyz=-0.0043743 0 -0.354 rpy=0 0 0
- joint Body_: axis 0 0 0 -> (none)
- joint BogieLB_: axis 0 0 -1 -> 0 0 1; origin xyz=-0.5677 0.17 0.172 rpy=1.5708 0 0 -> xyz=-0.5677 0.171999375553972 -0.170000631790131 rpy=0 0 0
- joint BogieLF_: axis 1.2372E-05 0 -1 -> 0 0 1; origin xyz=0.34839 0.099747 -0.0373 rpy=1.5708 0 0 -> xyz=0.34839 -0.0373003663909378 -0.0997468629887767 rpy=0 0 0
- joint BogieLM_: axis 1.2372E-05 0 -1 -> 0 0 1; origin xyz=0.34839 0.099747 -0.0373 rpy=1.5708 0 0 -> xyz=-0.219193607208571 -0.0373003663909378 -0.0997468629887767 rpy=0 0 0
- joint BogieRB_: axis 0 0 -1 -> 0 0 1; origin xyz=-0.567962211834988 -0.355999999999961 -0.0669999619615883 rpy=0 0 0 -> xyz=-0.567695341834988 -0.171999999999961 -0.169999961961588 rpy=0 0 0; parent base_link -> RightMainRocket_Link
- joint BogieRF_: axis 1.2371927108521E-05 0 -0.999999999923468 -> 0 0 1; origin xyz=0.348391502430392 0.0997469619704544 0.0373000000042916 rpy=1.57079632689944 0 0 -> xyz=0.348391502430392 0.0372996336129902 -0.0997470989803318 rpy=0 0 0
- joint BogieRM_: axis 1.23718983585148E-05 0 -0.999999999923468 -> 0 0 1; origin xyz=-0.219194109044066 0.0997641738351368 0.0373000000077186 rpy=1.57079632685489 0 0 -> xyz=-0.219194109044066 0.0372996335531945 -0.0997643108450141 rpy=0 0 0
- joint IMU_: axis 0 0 0 -> (none)
- joint LeftMainRocket_: axis 0 0 -1 -> 0 1 0; limit lower=-0.4 upper=0.4 effort=0 velocity=1 -> lower=-0.4 upper=0.4 effort=10 velocity=1; origin xyz=-0.00026687 0.184 0.103 rpy=-1.5708 0 0 -> xyz=-0.00026687 0.184 0.103 rpy=0 0 0
- joint LeftViceRocket_: axis 0 0 1 -> 0 1 0; origin xyz=0.219100000001228 0.0702529999871935 0.209300000002482 rpy=0 0 0 -> xyz=0.219100000001228 0.209299741947392 -0.0702537687885477 rpy=0 0 0
- joint Lidar_: axis 0 0 0 -> (none)
- joint RightMainRocket_: axis 0 0 1 -> 0 1 0; limit lower=-0.4 upper=0.4 effort=0 velocity=1 -> lower=-0.4 upper=0.4 effort=10 velocity=1; origin xyz=-0.00026687 -0.184 0.103 rpy=-1.5708 0 0 -> xyz=-0.00026687 -0.184 0.103 rpy=0 0 0
- joint RightViceRocket_: axis 0 0 -1 -> 0 1 0; origin xyz=0.219099999998321 0.0702530000126312 -0.209299999997518 rpy=0 0 0 -> xyz=0.219099999998321 -0.209300258049784 -0.0702522312103291 rpy=0 0 0
- joint WheelLB_: axis 0 0 1 -> 0 1 0; origin xyz=0 0 -0.162 rpy=-1.5708 0 0 -> xyz=0 0 -0.162 rpy=0 0 0
- joint WheelLF_: axis 0 0 1 -> 0 1 0; origin xyz=0 0 -0.161999999985028 rpy=-1.5707963267052 0 0 -> xyz=0 0 -0.161999999985028 rpy=0 0 0
- joint WheelLM_: axis 0 0 1 -> 0 1 0; origin xyz=-0.567583607208571 0 -0.162017211837628 rpy=-1.5707963267652 0 0 -> xyz=0 0 -0.162017211837628 rpy=0 0 0
- joint WheelRB_: axis 0 0 -1 -> 0 1 0; origin xyz=0 0 -0.162 rpy=-1.5708 0 0 -> xyz=0 0 -0.162 rpy=0 0 0
- joint WheelRF: axis 0 0 -1 -> 0 1 0; origin xyz=0 0 -0.16199999998823 rpy=-1.57079632689944 0 0 -> xyz=0 -5.95042290663095e-07 -0.161999999987137 rpy=0 0 0
- joint WheelRM_: axis 0 0 -1 -> 0 1 0; origin xyz=0 0 -0.161999999990611 rpy=-1.57079632685489 0 0 -> xyz=0 -5.95049507778889e-07 -0.161999999989518 rpy=0 0 0
- joint ZED_: axis 0 0 0 -> (none)
